File: PCB/LED.kicad_sch (KiCad schematic)
At the start: 11 parts

Commit message: PCB作成（続き）
Connections:
- no-connect marks 0 -> 1
Changed lines of the file:
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@@
 		)
+	)
+	(no_connect
+		(at 182.88 31.75)
 	)
 	(wire
