File: PCB/macro-keyboard.kicad_pcb (KiCad board)
At the start: 2 copper layers, 100 x 40 mm, 35 parts, among them P1 USB_C_Plug_USB2.0, SW1 DFU-mode, SW10 keySW, SW11 DFU-mode, SW2 RotaryEncoder, SW3 keySW, SW4 keySW, SW5 keySW, SW6 keySW, SW7 keySW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

Commit message: PCB作成
Parts:
- removed D1: SK6812MINI-E, LED_SMD:LED_SK6812MINI-E_3.2x2.8mm_P1.5mm_ReverseMount
- added C5: 0.1u, Capacitor_SMD:C_0603_1608Metric_Pad1.08x0.95mm_HandSolder, B.Cu at (131.3, 136.1)
- added C6: 3.9u, Capacitor_SMD:C_0603_1608Metric_Pad1.08x0.95mm_HandSolder, B.Cu at (131.3, 138.9)
- added D11: WS2812B, LED_SMD:LED_WS2812B_PLCC4_5.0x5.0mm_P3.2mm, B.Cu at (130.8, 132.3)
- added D12: WS2812B, LED_SMD:LED_WS2812B_PLCC4_5.0x5.0mm_P3.2mm, B.Cu at (96.7, 132.0)
- added D13: WS2812B, LED_SMD:LED_WS2812B_PLCC4_5.0x5.0mm_P3.2mm, B.Cu at (55.0, 140.5)
- added D14: WS2812B, LED_SMD:LED_WS2812B_PLCC4_5.0x5.0mm_P3.2mm, B.Cu at (55.2, 157.1)
- added D15: WS2812B, LED_SMD:LED_WS2812B_PLCC4_5.0x5.0mm_P3.2mm, B.Cu at (72.5, 163.4)
- added D16: WS2812B, LED_SMD:LED_WS2812B_PLCC4_5.0x5.0mm_P3.2mm, B.Cu at (98.6, 163.6)
- added D17: WS2812B, LED_SMD:LED_WS2812B_PLCC4_5.0x5.0mm_P3.2mm, B.Cu at (129.2, 163.6)
- added D18: WS2812B, LED_SMD:LED_WS2812B_PLCC4_5.0x5.0mm_P3.2mm, B.Cu at (146.8, 156.9)
- added D19: WS2812B, LED_SMD:LED_WS2812B_PLCC4_5.0x5.0mm_P3.2mm, B.Cu at (147.3, 139.2)
- C1, C2, C3, C4, R1, R2, R3, R4: moved to B.Cu
- D2, D3, D4, D5, D6, D7, D8, D9: moved to F.Cu
- moved D9 117.1 mm to (142.2, 157.5), turned to 180 degrees
- moved U1 116.5 mm to (78.8, 143.0)
- moved D8 116.1 mm to (142.2, 160.0), turned to 180 degrees
- moved D7 115.2 mm to (142.2, 162.6), turned to 180 degrees
- moved D6 114.2 mm to (142.2, 165.1), turned to 180 degrees
- moved D5 108.0 mm to (142.5, 131.6), turned to 180 degrees
- moved D4 107.0 mm to (142.5, 134.1), turned to 180 degrees
- moved D3 106.0 mm to (142.5, 136.7), turned to 180 degrees
- moved D2 105.0 mm to (142.5, 139.2), turned to 180 degrees
- moved SW3 93.3 mm to (66.0, 138.7), turned to 90 degrees
- moved SW6 93.3 mm to (123.2, 138.7)
- moved SW8 93.3 mm to (85.1, 157.7)
- moved SW9 93.3 mm to (104.1, 157.7)
- moved SW10 93.3 mm to (123.2, 157.7)
- moved SW5 93.3 mm to (104.1, 138.7)
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
Commit message: PCB作成（続き）
Parts:
- removed P1: USB_C_Plug_USB2.0, Connector_USB:USB_C_Receptacle_GCT_USB4105-xx-A_16P_TopMnt_Horizontal
- removed R1, R2: 5.1k, Resistor_SMD:R_0603_1608Metric_Pad0.98x0.95mm_HandSolder
- added J1: USB_C_Receptacle_USB2.0_16P, Connector_USB:USB_C_Receptacle_GCT_USB4105-xx-A_16P_TopMnt_Horizontal, B.Cu at (73.9, 132.1)
- added R5: 5.1k, Resistor_SMD:R_0603_1608Metric_Pad0.98x0.95mm_HandSolder, B.Cu at (70.2, 141.2)
- added R6: 5.1k, Resistor_SMD:R_0603_1608Metric_Pad0.98x0.95mm_HandSolder, B.Cu at (70.2, 138.7)
- SW2: footprint Rotary_Encoder:RotaryEncoder_Alps_EC12E-Switch_Vertical_H20mm -> Rotary_Encoder:RotaryEncoder_Alps_EC12E_Vertical_H20mm
- moved C4 3.81 mm to (98.3, 136.7)
- moved R4 3.81 mm to (94.7, 136.7), turned to 180 degrees
- moved C1 3.30 mm to (80.9, 138.2)
- moved C2 2.29 mm to (80.9, 135.4)
- moved C3 2.18 mm to (114.6, 140.2)
- moved R3 2.18 mm to (114.6, 137.7)
- moved U1 1.15 mm to (78.7, 144.1)
- moved D18 1.02 mm to (147.7, 156.4)
- moved D19 0.90 mm to (147.8, 140.0), turned to -90 degrees
- moved SW2 0.60 mm to (135.2, 145.7)
- moved D11 0.51 mm to (130.3, 132.3)
- turned C5 to 180 degrees
- turned C6 to 180 degrees
- turned SW8 to 180 degrees
Routing:
- net +5V: track 0.00 -> 268.4 mm
- net GND: track 0.00 -> 196.2 mm
- net Net-(D12-DOUT): track 0.00 -> 44.6 mm
- net Net-(D11-DOUT): track 0.00 -> 34.1 mm
- net Net-(D16-DOUT): track 0.00 -> 27.1 mm
- net Net-(D15-DOUT): track 0.00 -> 23.5 mm
- net /D-: track 0.00 -> 22.9 mm
- net Net-(D14-DOUT): track 0.00 -> 22.5 mm
- net Net-(D17-DOUT): track 0.00 -> 21.5 mm
- net Net-(D13-DOUT): track 0.00 -> 13.2 mm
- net /D+: track 0.00 -> 13.1 mm
- net Net-(D18-DOUT): track 0.00 -> 12.8 mm
- net +3V3: track 0.00 -> 5.51 mm

Commit message: 配線
Parts:
- moved C5 0.76 mm to (130.6, 136.1)
- moved D11 0.51 mm to (129.8, 132.3)
- moved C6 0.25 mm to (131.1, 138.9)
Routing:
- net Net-(D2-A): track 0.00 -> 78.3 mm
- net Net-(D3-A): track 0.00 -> 57.6 mm
- net Net-(D4-A): track 0.00 -> 32.0 mm
- net /debug: track 0.00 -> 23.5 mm, vias 0 -> 2
- net Net-(D5-A): track 0.00 -> 12.8 mm
- net /Row0: track 0.00 -> 9.62 mm, vias 0 -> 1
- net /Row1: track 0.00 -> 9.55 mm, vias 0 -> 1
- net /LED: track 0.00 -> 9.35 mm
- net Net-(J1-CC2): track 0.00 -> 9.04 mm, vias 0 -> 2
- net Net-(J1-CC1): track 0.00 -> 3.59 mm
- net /D-: track 22.9 -> 24.0 mm

Commit message: PCB作成
Parts:
- added G***: LOGO, sakura:sakura, F.Cu at (127.5, 88.2)
- added G***: LOGO, silkscreen:redstone, B.Cu at (102.5, 103.3)
- moved C3 73.0 mm to (150.6, 76.7)
- moved D12 73.0 mm to (132.8, 68.5)
- moved D17 73.0 mm to (165.3, 100.1)
- moved D18 73.0 mm to (183.8, 92.9)
- moved D19 73.0 mm to (183.9, 76.5)
- moved D2 73.0 mm to (178.6, 75.7)
- moved D4 73.0 mm to (178.6, 70.6)
- moved D5 73.0 mm to (178.6, 68.1)
- moved D8 73.0 mm to (178.3, 96.5)
- moved H5 73.0 mm to (130.7, 84.7)
- moved J1 73.0 mm to (110.0, 68.6)
- moved R3 73.0 mm to (150.6, 74.2)
- moved SW10 73.0 mm to (159.3, 94.2)
- moved SW2 73.0 mm to (171.2, 82.2)
- moved SW6 73.0 mm to (159.3, 75.2)
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Routing:
- net GND: track 196.2 -> 330.2 mm, vias 0 -> 268
- net /Row0: track 9.62 -> 95.9 mm, vias 1 -> 3
- net Net-(D6-A): track 0.00 -> 82.2 mm
- net /Row1: track 9.55 -> 88.5 mm, vias 1 -> 3
- net /rotary-A: track 0.00 -> 70.6 mm, vias 0 -> 2
- net /rotary-B: track 0.00 -> 67.5 mm, vias 0 -> 2
- net /LED: track 9.35 -> 64.8 mm, vias 0 -> 2
- net /Col3: track 0.00 -> 53.1 mm, vias 0 -> 2
- net /D+: track 13.1 -> 64.1 mm, vias 0 -> 2
- net +3V3: track 5.51 -> 53.9 mm, vias 0 -> 4
- net Net-(D8-A): track 0.00 -> 46.9 mm
- net /Col0: track 0.00 -> 44.2 mm
- net Net-(D7-A): track 0.00 -> 43.8 mm
- net /Col2: track 0.00 -> 35.1 mm, vias 0 -> 2
- net /Col1: track 0.00 -> 29.2 mm, vias 0 -> 2
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- added copper zone on B.Cu, net GND
- added copper zone on F.Cu, net GND
Other:
- board text added: "DEBUG"
- board text added: "DFU"
- board text added: "USB接続"
- board text added: "ch552t"
- board text added: "designed by 2k2e2n"

Commit message: 完成
Parts:
- added QR*****: qrcode, QRcode:qrcode, B.Cu at (149.7, 96.5)
- moved R3 0.47 mm to (150.6, 73.7)
Routing:
- net /D-: track 23.2 -> 21.7 mm
- net /D+: track 64.1 -> 64.8 mm
- net GND: vias 268 -> 271
Other:
- board text added: "2026/05/14"
- board text added: "V1.0"
- board text added: "ch552T"
- board text added: "macro-key SAKURA"
- board text removed: "ch552t"
