File: PCB/macro-keyboard.kicad_sch (KiCad schematic)
At the start: 0 parts

Commit message: 回路図完成
Parts:
- added C1, C2, C3, C4: 0.1u, Capacitor_SMD:C_0603_1608Metric_Pad1.08x0.95mm_HandSolder, symbol Device:C
- added D1: SK6812MINI-E, LED_SMD:LED_SK6812MINI-E_3.2x2.8mm_P1.5mm_ReverseMount, symbol LED:SK6812MINI-E
- added D2, D3, D4, D5, D6, D7, D8, D9: D, Diode_THT:D_DO-35_SOD27_P7.62mm_Horizontal, symbol Device:D
- added H1, H2, H3, H4, H5: MountingHole, MountingHole:MountingHole_3.2mm_M3, symbol Mechanical:MountingHole
- added P1: USB_C_Plug_USB2.0, Connector_USB:USB_C_Receptacle_GCT_USB4105-xx-A_16P_TopMnt_Horizontal, symbol Connector:USB_C_Plug_USB2.0
- added R1, R2: 5.1k, Resistor_SMD:R_0603_1608Metric_Pad0.98x0.95mm_HandSolder, symbol Device:R
- added R3, R4: 10k, Resistor_SMD:R_0603_1608Metric_Pad0.98x0.95mm_HandSolder, symbol Device:R
- added SW1, SW11: DFU-mode, Button_Switch_SMD:SW_SPST_EVQP0, symbol Switch:SW_Push
- added SW10, SW3, SW4, SW5, SW6, SW7, SW8, SW9: keySW, PCM_Switch_Keyboard_Hotswap_Kailh:SW_Hotswap_Kailh_MX_Plated_1.00u, symbol Switch:SW_Push
- added SW2: RotaryEncoder, Rotary_Encoder:RotaryEncoder_Alps_EC12E-Switch_Vertical_H20mm, symbol Device:RotaryEncoder
- added U1: CH552T, Package_SO:TSSOP-20_4.4x6.5mm_P0.65mm, symbol macrokey:ch552t
Connections:
- new net: P1.A5 (CC), R1.1, R2.1
- new net: C3.2, R3.1, SW1.1
- new net: D9.2 (A), SW10.1
- new net: D3.2 (A), SW4.1
- new net: D6.2 (A), SW7.1
- new net: D4.2 (A), SW5.1
- new net: D2.2 (A), SW3.1
- new net: D7.2 (A), SW8.1
- new net: D8.2 (A), SW9.1
- new net: D5.2 (A), SW6.1
- new net +3V3: C1.1, C3.1, SW1.2, U1.20 (V33)
- new net +5V: C2.1, D1.3 (VDD), P1.A4 (VBUS), P1.A9 (VBUS), P1.B4 (VBUS), P1.B9 (VBUS), R4.2, U1.19 (VCC/VDD)
- new net Col0: SW3.2, SW7.2, U1.4 (P1.6/MISO/RXD1/TIN4)
- new net Col1: SW4.2, SW8.2, U1.5 (P1.7/SCK/TXD1/TIN5)
- new net Col2: SW5.2, SW9.2, U1.6 (RST/T2EX_/CAP2_)
- new net Col3: SW10.2, SW6.2, U1.7 (P1.0/T2/CAP1/TIN0)
- new net D+: P1.A6 (D+), R3.2, U1.14 (P3.6/UDP)
- new net D-: P1.A7 (D-), U1.15 (P3.7/UDM)
- new net GND: C1.2, C2.2, C4.1, D1.1 (VSS), P1.A1 (GND), P1.A12 (GND), P1.B1 (GND), P1.B12 (GND), P1.SH (SHIELD), R1.2, R2.2, SW11.1, SW2.C, U1.18 (GND/VSS)
- new net LED: D1.2 (DIN), U1.9 (P3.1/PWM2_/TXD)
- new net Row0: D2.1 (K), D3.1 (K), D4.1 (K), D5.1 (K), U1.12 (P3.4/PWM2/RXD1_/T0)
- new net Row1: D6.1 (K), D7.1 (K), D8.1 (K), D9.1 (K), U1.11 (P3.3/INT1)
- new net debug: C4.2, R4.1, SW11.2, U1.10 (P3.0/PWM1_/RXD)
- new net rotary-A: SW2.A, U1.2 (P1.4/T2_/CAP1_/SCS/TIN2/UCC1/AIN1)
- new net rotary-B: SW2.B, U1.3 (P1.5/MOSI/PWM1/TIN3/UCC2/AIN2)
- no-connect marks 0 -> 7

Commit message: PCB作成
Parts:
- removed D1: SK6812MINI-E, LED_SMD:LED_SK6812MINI-E_3.2x2.8mm_P1.5mm_ReverseMount, symbol LED:SK6812MINI-E
Connections:
- no-connect marks 7 -> 6
Other:
- added sheet LED (LED.kicad_sch)

Commit message: PCB作成（続き）
Parts:
- removed P1: USB_C_Plug_USB2.0, Connector_USB:USB_C_Receptacle_GCT_USB4105-xx-A_16P_TopMnt_Horizontal, symbol Connector:USB_C_Plug_USB2.0
- removed R1, R2: 5.1k, Resistor_SMD:R_0603_1608Metric_Pad0.98x0.95mm_HandSolder, symbol Device:R
- added J1: USB_C_Receptacle_USB2.0_16P, Connector_USB:USB_C_Receptacle_GCT_USB4105-xx-A_16P_TopMnt_Horizontal, symbol Connector:USB_C_Receptacle_USB2.0_16P
- added R5, R6: 5.1k, Resistor_SMD:R_0603_1608Metric_Pad0.98x0.95mm_HandSolder, symbol Device:R
- SW2: footprint Rotary_Encoder:RotaryEncoder_Alps_EC12E-Switch_Vertical_H20mm -> Rotary_Encoder:RotaryEncoder_Alps_EC12E_Vertical_H20mm
Connections:
- net +5V: now also J1.A4 (VBUS), J1.A9 (VBUS), J1.B4 (VBUS), J1.B9 (VBUS)
- net D+: now also J1.A6 (D+), J1.B6 (D+)
- net D-: now also J1.A7 (D-), J1.B7 (D-)
- net GND: now also J1.A1 (GND), J1.A12 (GND), J1.B1 (GND), J1.B12 (GND), J1.SH (SHIELD), R5.2, R6.2
- new net: J1.A5 (CC1), R6.1
- new net: J1.B5 (CC2), R5.1
- no-connect marks 6 -> 7
Other:
- moved on the sheet: C1, C2, C3, R3, SW1, U1

Commit message: PCB作成
Other:
- title: (none) -> macro-key
Changed lines of the file:
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@@
 	(generator_version "10.0")
 	(paper "A4")
+	(title_block
+		(title "macro-key")
+		(date "2026-05-14")
+	)
 	(rectangle
 		(start 113.03 23.5344)

Commit message: 完成
Parts:
- SW11: value DFU-mode -> debug-SW
Changed lines of the file:
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@@
 			)
 		)
-		(property "Value" "DFU-mode"
+		(property "Value" "debug-SW"
 			(at 139.192 48.26 0)
 			(show_name no)

Commit message: ソフトウェアを作成
Other:
- note added: "2.2k"
- note added: "memo col2がリセットピンに接続されている⇒P3.2で代用 BOOTするとき、10kだと大きすぎて書き込めない OSTW3535C1のパッケージサイズ違う 上のLED使うならVCCを3v3にする"
Changed lines of the file:
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@@
+		)
+	)
+	(text "2.2k"
+		(exclude_from_sim no)
+		(at 90.17 188.468 0)
+		(effects
+			(font
+				(size 1.27 1.27)
+			)
+		)
+	)
+	(text "memo\ncol2がリセットピンに接続されている⇒P3.2で代用\nBOOTするとき、10kだと大きすぎて書き込めない\nOSTW3535C1のパッケージサイズ違う\n上のLED使うならVCCを3v3にする"
+		(exclude_from_sim no)
+		(at 95.758 102.362 0)
+		(effects
+			(font
+				(size 1.27 1.27)
+			)
 		)
 	)
@@
 		)
 	)
+	(polyline
+		(pts
+			(xy 85.09 184.15) (xy 85.09 185.42)
+		)
+		(stroke
+			(width 0)
+			(type default)
+		)
+	)
 	(wire
 		(pts
@@
 		)
 	)
+	(polyline
+		(pts
+			(xy 85.09 184.15) (xy 85.09 185.42)
+		)
+		(stroke
+			(width 0)
+			(type default)
+		)
+	)
 	(wire
 		(pts
@@
 		)
 	)
+	(polyline
+		(pts
+			(xy 86.36 185.42) (xy 85.09 184.15)
+		)
+		(stroke
+			(width 0)
+			(type default)
+		)
+	)
 	(wire
 		(pts
@@
 		)
 	)
+	(polyline
+		(pts
+			(xy 85.09 184.15) (xy 86.36 184.15)
+		)
+		(stroke
+			(width 0)
+			(type default)
+		)
+	)
 	(wire
 		(pts
@@
 		)
 		(stroke
+			(width 0)
+			(type default)
+		)
+	)
+	(polyline
+		(pts
+			(xy 86.36 185.42) (xy 87.63 186.69)
+		)
+		(stroke
