File: case/Top-mount/macro-keyboard-case.kicad_pcb (KiCad board)
At the start: 2 copper layers, 100 x 40 mm, 16 parts, among them SW10 keySW, SW2 RotaryEncoder, SW3 keySW, SW4 keySW, SW5 keySW, SW6 keySW, SW7 keySW, SW8 keySW, SW9 keySW

Commit message: ケース設計
Parts:
- removed SW2: RotaryEncoder, Rotary_Encoder:RotaryEncoder_Alps_EC12E_Vertical_H20mm
